File: iw18-hs.kicad_pcb (KiCad board)
At the start: 2 copper layers, 217.7 x 30 mm, 139 parts, among them J2 Conn_02x10_Counter_Clockwise, J3 Conn_02x10_Counter_Clockwise, J4 Conn_02x08_Odd_Even, J5 Conn_02x08_Odd_Even, J6 Conn_01x04_MountingPin, J7 Conn_01x04_MountingPin, J8 USB_C_Receptacle_USB2.0_16P, Q1 Q_NMOS_GSD, Q2 Q_NMOS_GDS, SW1 SW_SPST, SW2 SW_SPDT, SW3 SLLB120200, U1 IV-18, U10 TXS0104EPW, U11 MAX811TEUS-T, U12 AT24CS08-STUM, U13 MQ-6, U14 BME680, U15 LSM6DS3, U16 74LVC1G125, U17 USBLC6-2P6, U18 USBLC6-2P6, U19 PCF8574RGTR, U2 BQ25895RTW, U20 TMUX154ERSW, U3 ESP32-C6-WROOM-1, U4 LM1117DT-3.3, U5 MCP4017-xxxxLT, U6 TPS25751DREFR_C30169739, U7 LM3478MA, U8 USBLC6-2P6, U9 DRV8837

Commit message: Plan power planes
Parts:
- added C5: 47uF, Capacitor_SMD:C_0805_2012Metric, F.Cu at (163.0, 96.4)
- moved R17 64.3 mm to (193.7, 114.7), turned to 180 degrees
- moved R18 60.1 mm to (190.2, 114.7), turned to 0 degrees
- moved R19 33.4 mm to (184.0, 97.2), turned to 0 degrees
- moved R5 16.5 mm to (237.9, 94.3), turned to -90 degrees
- moved C50 16.5 mm to (245.7, 111.0), turned to 180 degrees
- moved Q1 15.4 mm to (241.4, 93.8), turned to 90 degrees
- moved R4 13.6 mm to (241.9, 111.0), turned to 0 degrees
- moved C48 13.2 mm to (228.9, 114.7)
- moved C49 13.2 mm to (228.9, 107.5)
- moved U14 13.2 mm to (233.8, 111.1)
- moved U15 13.2 mm to (228.8, 111.2)
- moved C46 13.2 mm to (233.9, 114.5)
- moved C47 13.2 mm to (233.7, 107.5)
- moved C41 3.02 mm to (125.5, 103.1), turned to 90 degrees
- moved C40 2.39 mm to (144.9, 103.1)
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Routing:
- added copper zone on In1.Cu, net +3.3V
- added copper zone on In1.Cu, net +3.3VA
- added copper zone on In1.Cu, net +5V
- added copper zone on In2.Cu, net GND
- added copper zone on In1.Cu, net VBUS
Other:
- outline, holes or cut-outs redrawn
- copper layers 2 -> 4

Commit message: Start routing
Parts:
- moved C33 19.7 mm to (107.8, 115.5), turned to 0 degrees
- moved R18 18.9 mm to (207.9, 108.1), turned to 90 degrees
- moved R17 17.5 mm to (209.9, 108.1), turned to 90 degrees
- moved U9 15.9 mm to (104.3, 114.7)
- moved C45 12.1 mm to (115.6, 96.1), turned to 0 degrees
- moved R3 11.2 mm to (142.3, 84.9), turned to 0 degrees
- moved C39 10.8 mm to (170.8, 96.0), turned to 90 degrees
- moved R2 8.54 mm to (143.1, 101.8)
- moved C40 7.06 mm to (148.7, 97.1), turned to 180 degrees
- moved R19 6.91 mm to (177.1, 97.3), turned to 180 degrees
- moved C41 6.68 mm to (128.5, 97.1), turned to 180 degrees
- moved R29 3.56 mm to (184.1, 97.3)
- moved R30 3.56 mm to (180.7, 97.3)
- moved C35 3.43 mm to (143.6, 94.4)
- moved C37 3.43 mm to (147.6, 94.4)
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Connections:
- U17 pad 1: Net-(J6-Pin_1) -> UART0_TX
- U17 pad 3: Net-(J6-Pin_2) -> UART0_RX
- U17 pad 4: UART0_RX -> Net-(J6-Pin_2)
- U17 pad 6: UART0_TX -> Net-(J6-Pin_1)
- U18 pad 1: Net-(J7-Pin_1) -> UART1_TX
- U18 pad 3: Net-(J7-Pin_2) -> UART1_RX
- U18 pad 4: UART1_RX -> Net-(J7-Pin_2)
- U18 pad 6: UART1_TX -> Net-(J7-Pin_1)
Routing:
- net SCL: track 0.00 -> 123.1 mm, vias 0 -> 8
- net SDA: track 0.00 -> 123.0 mm, vias 0 -> 8
- net Net-(U10-A4): track 0.00 -> 109.1 mm, vias 0 -> 2
- net Net-(U10-A1): track 0.00 -> 106.7 mm, vias 0 -> 2
- net Net-(U10-A2): track 0.00 -> 106.5 mm, vias 0 -> 2
- net Net-(U10-A3): track 0.00 -> 106.2 mm, vias 0 -> 2
- net Net-(J7-Pin_1): track 0.00 -> 90.9 mm, vias 0 -> 2
- net Net-(J7-Pin_2): track 0.00 -> 90.3 mm, vias 0 -> 2
- net PROGRAM_PD_CONTROLLER: track 0.00 -> 83.2 mm, vias 0 -> 2
- net Net-(U3-GPIO3/ADC1_CH3): track 0.00 -> 74.8 mm, vias 0 -> 2
- net Net-(J6-Pin_2): track 0.00 -> 74.6 mm, vias 0 -> 2
- net Net-(J6-Pin_1): track 0.00 -> 72.2 mm, vias 0 -> 2
- net USB_D+: track 0.00 -> 63.7 mm, vias 0 -> 2
- net USB_D-: track 0.00 -> 63.1 mm, vias 0 -> 2
- net CHG_INT: track 0.00 -> 59.3 mm, vias 0 -> 3
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