File: iw18-hs.kicad_pcb (KiCad board)
At the start: 4 copper layers, 217.7 x 30 mm, 140 parts, among them J2 Conn_02x10_Counter_Clockwise, J3 Conn_02x10_Counter_Clockwise, J4 Conn_02x08_Odd_Even, J5 Conn_02x08_Odd_Even, J6 Conn_01x04_MountingPin, J7 Conn_01x04_MountingPin, J8 USB_C_Receptacle_USB2.0_16P, Q1 Q_NMOS_GSD, Q2 Q_NMOS_GDS, SW1 SW_SPST, SW2 SW_SPDT, SW3 SLLB120200, U1 IV-18, U10 TXS0104EPW, U11 MAX811TEUS-T, U12 AT24CS08-STUM, U13 MQ-6, U14 BME680, U15 LSM6DS3, U16 74LVC1G125, U17 USBLC6-2P6, U18 USBLC6-2P6, U19 PCF8574RGTR, U2 BQ25895RTW, U20 TMUX154ERSW, U3 ESP32-C6-WROOM-1, U4 LM1117DT-3.3, U5 MCP4017-xxxxLT, U6 TPS25751DREFR_C30169739, U7 LM3478MA, U8 USBLC6-2P6, U9 DRV8837

Commit message: Route some
Parts:
- added JP1: SolderJumper_2_Open, Jumper:SolderJumper-2_P1.3mm_Open_RoundedPad1.0x1.5mm, F.Cu at (104.1, 96.4)
- added JP2: SolderJumper_2_Open, Jumper:SolderJumper-2_P1.3mm_Open_RoundedPad1.0x1.5mm, F.Cu at (88.7, 93.7)
- moved R15 23.7 mm to (121.3, 99.8), turned to -90 degrees
- moved TP4 20.6 mm to (135.5, 88.2)
- moved R16 17.2 mm to (125.6, 99.8), turned to -90 degrees
- moved TP7 16.8 mm to (229.0, 99.6)
- moved C50 15.1 mm to (245.7, 95.9), turned to 0 degrees
- moved R4 15.0 mm to (229.0, 103.3), turned to -90 degrees
- moved D2 14.4 mm to (144.4, 102.5), turned to 0 degrees
- moved R20 13.9 mm to (150.1, 88.7)
- moved C2 13.4 mm to (152.0, 88.7), turned to 90 degrees
- moved TP6 11.8 mm to (143.7, 97.7)
- moved R33 11.7 mm to (141.1, 96.6), turned to 90 degrees
- moved R3 7.96 mm to (146.7, 91.5)
- moved C47 7.60 mm to (236.8, 114.5)
- moved R34 7.48 mm to (170.7, 106.0), turned to 0 degrees
- moved C1 7.45 mm to (167.0, 97.1)
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Connections:
- net Net-(F1-Pad1) renamed VBUS_FUSED
- J2 pad 2: HEATER_A -> HEATER_B
- J2 pad 4: HEATER_B -> HEATER_A
- J3 pad 2: HEATER_A -> HEATER_B
- J3 pad 4: HEATER_B -> HEATER_A
- J6 pad 4: +5V -> Net-(J6-Pin_4)
- J7 pad 4: +5V -> Net-(J7-Pin_4)
- U19 pad 12: unconnected-(U19-P6-Pad12) -> PROGRAM_PD_CONTROLLER
- U19 pad 5: JOYSTICK_PUSH -> JOYSTICK_CCW1
- U19 pad 7: JOYSTICK_CCW1 -> JOYSTICK_PUSH
- U3 pad 23: PROGRAM_PD_CONTROLLER -> F_EN
- U3 pad 7: unconnected-(U3-MTDO/GPIO7-Pad7) -> F_PWM
- U3 pad 8: IMU_INT0 -> ETANOL_SENSE_ADC
- U3 pad 9: ETANOL_SENSE_ADC -> IMU_INT0
Routing:
- net GND: track 3.39 -> 210.7 mm, vias 4 -> 153
- net F_EN: track 0.00 -> 112.0 mm, vias 0 -> 4
- net F_PWM: track 0.00 -> 93.8 mm, vias 0 -> 4
- net +3.3V: track 4.48 -> 73.8 mm, vias 5 -> 19
- net HEATER_B: track 0.00 -> 68.0 mm, vias 0 -> 1
- net ETANOL_SENSE_ADC: track 0.00 -> 67.0 mm, vias 0 -> 2
- net IMU_INT0: track 0.00 -> 61.7 mm, vias 0 -> 3
- net SCL: track 123.1 -> 183.1 mm, vias 8 -> 12
- net SDA: track 123.0 -> 179.2 mm, vias 8 -> 14
- net ETANOL_SENSOR_HEAT: track 0.00 -> 54.6 mm, vias 0 -> 3
- net VPP: track 0.00 -> 53.7 mm, vias 0 -> 1
- net /VFD/D1: track 0.00 -> 52.4 mm, vias 0 -> 2
- net /VFD/A: track 0.00 -> 50.5 mm, vias 0 -> 1
- net /VFD/G: track 0.00 -> 50.3 mm, vias 0 -> 2
- net +5V: track 0.00 -> 49.5 mm, vias 0 -> 14
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
Commit message: Fix bridged trace
Parts:
- moved R33 0.51 mm to (141.6, 96.6)
Routing:
- net +3.3V: track 73.8 -> 94.9 mm, vias 19 -> 23
- net Net-(U11-~{RESET}): track 27.6 -> 35.1 mm
- net GND: track 210.7 -> 215.7 mm, vias 153 -> 156
- net USB_D+: track 63.7 -> 66.6 mm
- net USB_D-: track 63.1 -> 65.3 mm, vias 2 -> 4
- net Net-(SW1-B): track 27.0 -> 28.8 mm
- net unconnected-(RV4-Pad3): track 0.00 -> 0.58 mm
Other:
- board size 217.7 x 30 mm -> 217.7 x 30.5 mm
