File: power.kicad_sch (KiCad schematic)
At the start: 54 parts, among them J8 USB_C_Receptacle_USB2.0_16P, Q2 Q_NMOS_GDS, SW2 SW_SPDT, U16 74LVC1G125, U2 BQ25895RTW, U4 LM1117DT-3.3, U5 MCP4017-xxxxLT, U7 LM3478MA

Commit message: Start routing
Other:
- moved on the sheet: F1, J8, R15, R16, R3, TP3

Commit message: Route some
Connections:
- net VBUS_FUSED: now reaches F1.1, J8.A4 (VBUS), J8.A9 (VBUS), J8.B4 (VBUS), J8.B9 (VBUS)
Changed lines of the file:
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@@
+	)
+	(junction
+		(at 44.45 30.48)
+		(diameter 0)
+		(color 0 0 0 0)
 	)
 	(junction
@@
 	(wire
 		(pts
+			(xy 44.45 30.48) (xy 45.72 30.48)
+		)
+		(stroke
+			(width 0)
+			(type default)
+		)
+	)
+	(wire
+		(pts
 			(xy 149.86 24.13) (xy 151.13 24.13)
 		)
@@
 	(wire
 		(pts
+			(xy 44.45 20.32) (xy 44.45 30.48)
+		)
+		(stroke
+			(width 0)
+			(type default)
+		)
+	)
+	(wire
+		(pts
 			(xy 53.34 30.48) (xy 57.15 30.48)
 		)
@@
 	(wire
 		(pts
-			(xy 43.18 30.48) (xy 45.72 30.48)
+			(xy 43.18 30.48) (xy 44.45 30.48)
 		)
 		(stroke
@@
 		(pts
 			(xy 167.64 53.34) (xy 167.64 43.18)
+		)
+		(stroke
+			(width 0)
+			(type default)
+		)
+	)
+	(wire
+		(pts
+			(xy 36.83 20.32) (xy 44.45 20.32)
 		)
 		(stroke
@@
 			)
 		)
+	)
+	(global_label "VBUS_FUSED"
+		(shape input)
+		(at 36.83 20.32 180)
+		(fields_autoplaced yes)
+		(effects
+			(font
+				(size 1.27 1.27)
+			)
+			(justify right)
+		)
+		(property "Intersheetrefs" "${INTERSHEET_REFS}"
+			(at 21.931 20.32 0)
+			(hide yes)
+			(show_name no)
+			(do_not_autoplace no)
+			(effects
+				(font
+					(size 1.27 1.27)
+				)
+				(justify right)
+			)
+		)
